Commit message: I modified the Gazebo collision/surface properties of the rx200 robot in order to allow me to pickup items in Gazebo. Before these changes, the robot's finger's would close on an object and it would just slip.

File: interbotix_descriptions/urdf/rx200.urdf.xacro (robot description, xacro)
@@ -398,4 +398,102 @@
         </inertial>
       </link>
+     <gazebo reference="rx200/right_finger_link">
+       <collision>
+	<surface>
+          <friction>
+            <ode>
+              <mu>5000</mu>
+              <mu2>5000</mu2>
+              <fdir1>0 0 0</fdir1>
+      		<minDepth>0.003</minDepth>
+    		<maxVel>0</maxVel>
+      	</ode>
+            <torsional>
+              <coefficient>1</coefficient>
+              <patch_radius>0</patch_radius>
+              <surface_radius>0</surface_radius>
+              <use_patch_radius>1</use_patch_radius>
+              <ode>
+                <slip>0.1</slip>
+              </ode>
+            </torsional>
+          </friction>
+          <bounce>
+            <restitution_coefficient>0</restitution_coefficient>
+            <threshold>1e+06</threshold>
+          </bounce>
+          <contact>
+            <collide_without_contact>0</collide_without_contact>
+            <collide_without_contact_bitmask>1</collide_without_contact_bitmask>
+            <collide_bitmask>1</collide_bitmask>
+            <ode>
+              <soft_cfm>0</soft_cfm>
+              <soft_erp>0.2</soft_erp>
+              <kp>1e+13</kp>
+              <kd>1</kd>
+              <max_vel>0.01</max_vel>
+              <min_depth>0</min_depth>
+            </ode>
+            <bullet>
+              <split_impulse>1</split_impulse>
+              <split_impulse_penetration_threshold>-0.01</split_impulse_penetration_threshold>
+              <soft_cfm>0</soft_cfm>
+              <soft_erp>0.2</soft_erp>
+              <kp>1e+13</kp>
+              <kd>1</kd>
+            </bullet>
+          </contact>
+        </surface>
+        </collision>
+     </gazebo>
+     <gazebo reference="rx200/left_finger_link">
+       <collision>
+        <surface>
+          <friction>
+            <ode>
+              <mu>50000</mu>
+              <mu2>5000</mu2>
+              <fdir1>0 0 0</fdir1>
+      		<minDepth>0.003</minDepth>
+		    <maxVel>0</maxVel>
+      		</ode>
+            <torsional>
+              <coefficient>1</coefficient>
+              <patch_radius>0</patch_radius>
+              <surface_radius>0</surface_radius>
+              <use_patch_radius>1</use_patch_radius>
+              <ode>
+                <slip>0.1</slip>
+              </ode>
+            </torsional>
+          </friction>
+          <bounce>
+            <restitution_coefficient>0</restitution_coefficient>
+            <threshold>1e+06</threshold>
+          </bounce>
+          <contact>
+            <collide_without_contact>0</collide_without_contact>
+            <collide_without_contact_bitmask>1</collide_without_contact_bitmask>
+            <collide_bitmask>1</collide_bitmask>
+            <ode>
+              <soft_cfm>0</soft_cfm>
+              <soft_erp>0.2</soft_erp>
+              <kp>1e+13</kp>
+              <kd>1</kd>
+              <max_vel>0.01</max_vel>
+              <min_depth>0</min_depth>
+            </ode>
+            <bullet>
+              <split_impulse>1</split_impulse>
+              <split_impulse_penetration_threshold>-0.01</split_impulse_penetration_threshold>
+              <soft_cfm>0</soft_cfm>
+              <soft_erp>0.2</soft_erp>
+              <kp>1e+13</kp>
+              <kd>1</kd>
+            </bullet>
+          </contact>
+        </surface>
+        </collision>
+     </gazebo>
     </xacro:if>
   </xacro:if>
